File: pcb/clock.brd (EAGLE design)
At the start: 76.2 x 25.4 mm, 23 parts, among them IC1 74AHCT125, U1 ESP-01, U2 LD1117V33

Commit message: Minor adjustments
Routing:
- net VCC: track 54.5 -> 47.3 mm
Changed lines of the file:
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@@
 </element>
 <element name="R1" library="rcl" package="0204/5" value="470" x="29.845" y="22.86" smashed="yes">
-<attribute name="VALUE" x="31.75" y="23.495" size="1.016" layer="27" ratio="10" rot="R180"/>
+<attribute name="VALUE" x="29.845" y="22.86" size="1.016" layer="27" ratio="10" rot="R180" align="center"/>
 </element>
 <element name="C4" library="rcl" package="E3,5-8" value="1000uF" x="71.12" y="5.08" smashed="yes" rot="R270">
@@
 </element>
 <element name="R2" library="rcl" package="0204/5" value="10K" x="39.37" y="5.08" smashed="yes" rot="R270">
-<attribute name="VALUE" x="38.735" y="6.985" size="1.016" layer="27" ratio="10" rot="R270"/>
+<attribute name="VALUE" x="39.37" y="5.08" size="1.016" layer="27" ratio="10" rot="R270" align="center"/>
 </element>
 <element name="R3" library="rcl" package="0204/5" value="1.8K" x="4.445" y="20.32" smashed="yes" rot="R270">
-<attribute name="VALUE" x="3.81" y="22.225" size="1.016" layer="27" ratio="10" rot="R270"/>
+<attribute name="VALUE" x="4.445" y="20.32" size="1.016" layer="27" ratio="10" rot="R270" align="center"/>
 </element>
 <element name="R4" library="rcl" package="0204/5" value="3.3K" x="2.54" y="20.32" smashed="yes" rot="R90">
-<attribute name="VALUE" x="1.905" y="22.225" size="1.016" layer="27" ratio="10" rot="R270"/>
+<attribute name="VALUE" x="2.54" y="20.32" size="1.016" layer="27" ratio="10" rot="R270" align="center"/>
 </element>
 <element name="IC1" library="ic-package" package="DIL14" value="74AHCT125" x="24.13" y="16.51" smashed="yes" rot="R180">
@@
 <element name="S1" library="my-custom" package="TACTILE-BUTTON-MJTP1230" value="MJTP1230" x="9.525" y="11.43" rot="R180"/>
 <element name="R6" library="rcl" package="0204/5" value="10K" x="37.465" y="5.08" smashed="yes" rot="R270">
-<attribute name="VALUE" x="36.83" y="6.985" size="1.016" layer="27" ratio="10" rot="R270"/>
+<attribute name="VALUE" x="37.465" y="5.08" size="1.016" layer="27" ratio="10" rot="R270" align="center"/>
 </element>
 <element name="H1" library="holes" package="2,8-PAD" value="MOUNT-PAD-ROUND2.8" x="62.865" y="20.32"/>
@@
 <element name="D1" library="diode" package="DO41-7.6" value="1N5817-B" x="20.32" y="9.525" smashed="yes" rot="R180"/>
 <element name="R7" library="rcl" package="0204/5" value="10K" x="35.56" y="5.08" smashed="yes" rot="R270">
-<attribute name="VALUE" x="34.925" y="6.985" size="1.016" layer="27" ratio="10" rot="R270"/>
+<attribute name="VALUE" x="35.56" y="5.08" size="1.016" layer="27" ratio="10" rot="R270" align="center"/>
 </element>
 <element name="C5" library="rcl" package="C025-025X050" value="0.1uF" x="33.02" y="8.89" smashed="yes" rot="R270"/>
 <element name="R5" library="rcl" package="0204/5" value="1.8K" x="8.255" y="20.32" smashed="yes" rot="R270">
-<attribute name="VALUE" x="7.62" y="22.225" size="0.9906" layer="27" ratio="10" rot="R270"/>
+<attribute name="VALUE" x="8.255" y="20.32" size="0.9906" layer="27" ratio="10" rot="R270" align="center"/>
 </element>
 <element name="R8" library="rcl" package="0204/5" value="3.3K" x="6.35" y="20.32" smashed="yes" rot="R90">
-<attribute name="VALUE" x="5.715" y="22.225" size="0.9906" layer="27" ratio="10" rot="R270"/>
+<attribute name="VALUE" x="6.35" y="20.32" size="0.9906" layer="27" ratio="10" rot="R270" align="center"/>
 </element>
 </elements>
@@
 <wire x1="52.07" y1="21.58" x2="52.07" y2="19.05" width="1.016" layer="1"/>
 <wire x1="27.94" y1="2.54" x2="33.02" y2="2.54" width="1.016" layer="1"/>
-<wire x1="33.02" y1="2.54" x2="34.6075" y2="4.1275" width="1.016" layer="16"/>
-<wire x1="34.6075" y1="4.1275" x2="51.1175" y2="4.1275" width="1.016" layer="16"/>
 <wire x1="46.99" y1="20.32" x2="48.26" y2="19.05" width="1.016" layer="1"/>
 <wire x1="48.26" y1="19.05" x2="52.07" y2="19.05" width="1.016" layer="1"/>
-<wire x1="51.1175" y1="4.1275" x2="52.07" y2="5.08" width="1.016" layer="16"/>
-<wire x1="51.435" y1="5.715" x2="52.07" y2="5.08" width="0.4064" layer="1"/>
 <contactref element="R7" pad="2"/>
-<wire x1="35.56" y1="2.54" x2="33.02" y2="2.54" width="0.4064" layer="1"/>
-<wire x1="35.56" y1="2.54" x2="37.465" y2="2.54" width="0.4064" layer="1"/>
-<wire x1="37.465" y1="2.54" x2="39.37" y2="2.54" width="0.4064" layer="1"/>
+<wire x1="33.02" y1="2.54" x2="35.56" y2="2.54" width="1.016" layer="1"/>
+<wire x1="35.56" y1="2.54" x2="37.465" y2="2.54" width="1.016" layer="1"/>
+<wire x1="37.465" y1="2.54" x2="39.37" y2="2.54" width="1.016" layer="1"/>
+<wire x1="52.07" y1="5.08" x2="49.53" y2="2.54" width="1.016" layer="1"/>
+<wire x1="49.53" y1="2.54" x2="39.37" y2="2.54" width="1.016" layer="1"/>
 </signal>
 <signal name="+5V">
